File: Hardware/SparkFun_Simultaneous_RFID_Reader_M7E.brd (EAGLE design)
At the start: 35.6 x 61 mm, 77 parts, among them J5 U.FL, U1 UHF_RFID_NANO_MODULE_M7E_HECTO, U2 CH340C

Commit message: Fix DNP components and PROD_ID values
Parts:
- C1, C5, C8, C9: value 1.0pF -> DNP
Changed lines of the file:
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@@
 </element>
 <element name="E1" library="SparkFun-RF" package="TRACE_ANTENNA_915MHZ_THINGMAGIC" value="ANTENNA-GROUNDEDTRACE-915MHZ" x="30.48" y="43.18" smashed="yes" rot="R180"/>
-<element name="C1" library="SparkFun-Capacitors" package="0603" value="1.0pF" x="29.591" y="45.847" smashed="yes" rot="R180">
+<element name="C1" library="SparkFun-Capacitors" package="0603" value="DNP" x="29.591" y="45.847" smashed="yes" rot="R180">
 <attribute name="NAME" x="29.591" y="45.085" size="0.6096" layer="25" font="vector" ratio="20" rot="R180" align="bottom-center"/>
-<attribute name="PROD_ID" value="CAP-07879" x="29.591" y="45.847" size="1.778" layer="27" rot="R180" display="off"/>
+<attribute name="PROD_ID" value="" x="29.591" y="45.847" size="1.778" layer="27" rot="R180" display="off"/>
 <attribute name="VALUE" x="29.591" y="46.609" size="0.6096" layer="27" font="vector" ratio="20" rot="R180" align="top-center"/>
 </element>
@@
 <attribute name="VALUE" x="9.525" y="39.243" size="0.6096" layer="27" font="vector" ratio="20" align="top-left"/>
 </element>
-<element name="C5" library="SparkFun-Capacitors" package="0603" value="1.0pF" x="13.97" y="40.9321" smashed="yes" rot="R270">
+<element name="C5" library="SparkFun-Capacitors" package="0603" value="DNP" x="13.97" y="40.9321" smashed="yes" rot="R270">
 <attribute name="NAME" x="14.732" y="40.9321" size="0.6096" layer="25" font="vector" ratio="20" rot="R270" align="bottom-center"/>
-<attribute name="PROD_ID" value="CAP-07879" x="25.4" y="56.1721" size="1.778" layer="27" rot="R270" display="off"/>
+<attribute name="PROD_ID" value="" x="25.4" y="56.1721" size="1.778" layer="27" rot="R270" display="off"/>
 <attribute name="VALUE" x="13.208" y="40.9321" size="0.6096" layer="27" font="vector" ratio="20" rot="R270" align="top-center"/>
 </element>
@@
 <element name="R5" library="SparkFun-Resistors" package="0603" value="DNP" x="21.9202" y="41.783" smashed="yes">
 <attribute name="NAME" x="21.8948" y="42.545" size="0.6096" layer="25" font="vector" ratio="20" align="bottom-center"/>
-<attribute name="PROD_ID" value="RES-08609" x="21.8948" y="41.783" size="1.778" layer="27" display="off"/>
+<attribute name="PROD_ID" value="" x="21.8948" y="41.783" size="1.778" layer="27" display="off"/>
 <attribute name="VALUE" x="21.8948" y="41.021" size="0.6096" layer="27" font="vector" ratio="20" align="top-center"/>
 </element>
@@
 </element>
 <element name="U$8" library="output" package="UART0" value="" x="31.115" y="5.715" smashed="yes" rot="R90"/>
-<element name="C8" library="SparkFun-Capacitors" package="0603" value="1.0pF" x="19.05" y="40.9321" smashed="yes" rot="R270">
+<element name="C8" library="SparkFun-Capacitors" package="0603" value="DNP" x="19.05" y="40.9321" smashed="yes" rot="R270">
 <attribute name="NAME" x="19.812" y="40.9321" size="0.6096" layer="25" font="vector" ratio="20" rot="R270" align="bottom-center"/>
-<attribute name="PROD_ID" value="CAP-07879" x="19.05" y="40.9321" size="1.778" layer="27" rot="R270" display="off"/>
+<attribute name="PROD_ID" value="" x="19.05" y="40.9321" size="1.778" layer="27" rot="R270" display="off"/>
 <attribute name="VALUE" x="18.288" y="40.9321" size="0.6096" layer="27" font="vector" ratio="20" rot="R270" align="top-center"/>
 </element>
-<element name="C9" library="SparkFun-Capacitors" package="0603" value="1.0pF" x="26.67" y="40.9321" smashed="yes" rot="R270">
+<element name="C9" library="SparkFun-Capacitors" package="0603" value="DNP" x="26.67" y="40.9321" smashed="yes" rot="R270">
 <attribute name="NAME" x="27.432" y="40.9321" size="0.6096" layer="25" font="vector" ratio="20" rot="R270" align="bottom-center"/>
-<attribute name="PROD_ID" value="CAP-07879" x="26.67" y="40.9321" size="1.778" layer="27" rot="R270" display="off"/>
+<attribute name="PROD_ID" value="" x="26.67" y="40.9321" size="1.778" layer="27" rot="R270" display="off"/>
 <attribute name="VALUE" x="25.908" y="40.9321" size="0.6096" layer="27" font="vector" ratio="20" rot="R270" align="top-center"/>
 </element>
