File: Hardware/SparkFun_Simultaneous_RFID_Reader_M7E.sch (EAGLE design)
At the start: 43 parts, among them J5 U.FL, U1 UHF_RFID_NANO_MODULE_M7E_HECTO, U2 CH340C

Commit message: Design review updates
Add polygons to better fan out USB traces from ESD diode pads
Nudge R3 away from VOUT pad
Add VOUT range to schematic
Swap power LED and resistor for new version
Move via out of VO silk label
Nudge USB traces to get better GND pour around C7
Other:
- note added: "VOUT Range: Variable, nominally 3.3V while active. Typically 2.5V while idle."
Changed lines of the file:
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@@
 switch between internal
 and external antennas</text>
-<text x="12.7" y="106.68" size="1.27" layer="97" font="vector" align="center">VIN Range:
-3.3V - 5.5V</text>
+<text x="12.7" y="109.22" size="1.27" layer="97" font="vector" align="center">VOUT Range:
+Variable, nominally 3.3V
+while active. Typically
+2.5V while idle.</text>
 <text x="218.44" y="111.76" size="1.27" layer="97" font="vector" align="center">Cut PWR trace to
 remove power LED</text>
@@
 <text x="180.34" y="78.74" size="1.27" layer="97" font="vector" align="center">Use to switch between
 USB and serial header inputs</text>
+<text x="12.7" y="116.84" size="1.27" layer="97" font="vector" align="center">VIN Range:
+3.3V - 5.5V</text>
 </plain>
 <instances>

Commit message: Design review update
Actually update the power LED and resistor this time
Actually move the via on the VO silk this time
Actually nudge USB traces to get better GND pour around C7 this time
Parts:
- D2: device SparkFun-LED:LED-RED0603 -> SparkFun-LED:LED-RED_0603-KB
- R3: value 1k -> 4.7k; device SparkFun-Resistors:1KOHM-0603-1/10W-1% -> SparkFun-Resistors:4.7KOHM-0603-1/10W-1%
Changed lines of the file:
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@@
 <part name="S1" library="SparkFun-Switches" deviceset="SWITCH-DPDT" device="-SMD-AYZ0202"/>
 <part name="LOGO3" library="SparkFun-Aesthetics" deviceset="SFE_LOGO_NAME_FLAME" device=".2_INCH"/>
-<part name="D2" library="SparkFun-LED" deviceset="LED-RED" device="0603" value="Red"/>
+<part name="D2" library="SparkFun-LED" deviceset="LED-RED" device="_0603-KB" value="Red"/>
 <part name="PWR" library="SparkFun-Jumpers" deviceset="JUMPER-SMT_2_NC_TRACE" device="_SILK" package3d_urn="urn:adsk.eagle:package:39281/1"/>
-<part name="R3" library="SparkFun-Resistors" deviceset="1KOHM" device="-0603-1/10W-1%" value="1k"/>
+<part name="R3" library="SparkFun-Resistors" deviceset="4.7KOHM" device="-0603-1/10W-1%" value="4.7k"/>
 <part name="GND10" library="SparkFun-PowerSymbols" deviceset="GND" device=""/>
 <part name="C2" library="SparkFun-Capacitors" deviceset="10NF" device="-0603-50V-10%" value="10nF"/>

Commit message: Design review updates
Update section titles in schematic
Remote DTR and CTS silk from serial header
Add ordering instructions
Update measures
Parts:
- added LOGO4: SPECIAL_INSTRUCTIONS-ORDERING, SparkFun-Aesthetics:SPECIAL_INSTRUCTIONS-ORDERING
Other:
- note added: "UHF RFID Module - M7E Hecto"
- note added: "USB to UART - CH340"
- note removed: "M6E Nano"
- note removed: "USB to UART"
Changed lines of the file:
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@@
 <part name="GND22" library="SparkFun-PowerSymbols" deviceset="GND" device=""/>
 <part name="SUPPLY8" library="SparkFun-PowerSymbols" deviceset="V_USB" device=""/>
+<part name="LOGO4" library="SparkFun-Aesthetics" deviceset="SPECIAL_INSTRUCTIONS" device="-ORDERING"/>
 </parts>
 <sheets>
@@
 disconnect USB shield</text>
 <text x="45.72" y="180.34" size="2.54" layer="94" font="vector" align="center">USB Connector</text>
-<text x="139.7" y="180.34" size="2.54" layer="94" font="vector" align="center">USB to UART</text>
+<text x="137.16" y="180.34" size="2.54" layer="94" font="vector" align="center">USB to UART - CH340</text>
 <text x="215.9" y="180.34" size="2.54" layer="94" font="vector" align="center">Header Pins</text>
 <wire x1="0" y1="127" x2="96.52" y2="127" width="0.2032" layer="97" style="longdash"/>
@@
 <text x="114.3" y="68.58" size="2.54" layer="94" font="vector" align="center">Antennas</text>
 <wire x1="147.32" y1="63.5" x2="147.32" y2="76.2" width="0.2032" layer="97" style="longdash"/>
-<text x="40.64" y="121.92" size="2.54" layer="94" font="vector" align="center">M6E Nano</text>
+<text x="40.64" y="121.92" size="2.54" layer="94" font="vector" align="center">UHF RFID Module - M7E Hecto</text>
 <text x="180.34" y="121.92" size="2.54" layer="94" font="vector" align="center">UART Switch</text>
 <text x="88.9" y="43.18" size="1.27" layer="97" font="vector" align="center">Move 0 Ohm resistor to
@@
 <attribute name="VALUE" x="106.68" y="172.974" size="1.778" layer="96" align="bottom-center"/>
 </instance>
+<instance part="LOGO4" gate="G$1" x="226.06" y="33.02" smashed="yes"/>
 </instances>
 <busses>

Commit message: Fix DNP components and PROD_ID values
Parts:
- C1, C5, C8, C9: value 1.0pF -> DNP
Changed lines of the file:
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@@
 <part name="E1" library="SparkFun-RF" deviceset="ANTENNA-GROUNDED" device="TRACE-915MHZ"/>
 <part name="GND2" library="SparkFun-PowerSymbols" deviceset="GND" device=""/>
-<part name="C1" library="SparkFun-Capacitors" deviceset="1.0PF" device="-0603-50V-25%" value="1.0pF"/>
+<part name="C1" library="SparkFun-Capacitors" deviceset="1.0PF" device="-0603-50V-25%" value="DNP">
+<attribute name="PROD_ID" value=""/>
+</part>
 <part name="GND3" library="SparkFun-PowerSymbols" deviceset="GND" device=""/>
 <part name="L1" library="SparkFun-Coils" deviceset="3.9NH" device=""/>
@@
 <part name="SUPPLY13" library="SparkFun-PowerSymbols" deviceset="VIN" device=""/>
 <part name="J5" library="SparkFun-Connectors" deviceset="U.FL" device="" value="U.FL"/>
-<part name="C5" library="SparkFun-Capacitors" deviceset="1.0PF" device="-0603-50V-25%" value="1.0pF"/>
+<part name="C5" library="SparkFun-Capacitors" deviceset="1.0PF" device="-0603-50V-25%" value="DNP">
+<attribute name="PROD_ID" value=""/>
+</part>
 <part name="C6" library="SparkFun-Capacitors" deviceset="1.0NF/1000PF" device="-0603-50V-10%" value="1nF"/>
 <part name="GND16" library="SparkFun-PowerSymbols" deviceset="GND" device=""/>
@@
 <part name="GND18" library="SparkFun-PowerSymbols" deviceset="GND" device=""/>
 <part name="R4" library="SparkFun-Resistors" deviceset="0OHM" device="-0603-1/10W" value="0"/>
-<part name="R5" library="SparkFun-Resistors" deviceset="0OHM" device="-0603-1/10W" value="DNP"/>
+<part name="R5" library="SparkFun-Resistors" deviceset="0OHM" device="-0603-1/10W" value="DNP">
+<attribute name="PROD_ID" value=""/>
+</part>
 <part name="D3" library="SparkFun-IC-Power" deviceset="PRTR5V0U2" device="F"/>
 <part name="GND19" library="SparkFun-PowerSymbols" deviceset="GND" device=""/>
 <part name="J1" library="SparkFun-Connectors" deviceset="CONN_08" device="NO_SILK_DNP"/>
 <part name="J2" library="SparkFun-Connectors" deviceset="CONN_06" device="NO_SILK_NO_POP"/>
-<part name="C8" library="SparkFun-Capacitors" deviceset="1.0PF" device="-0603-50V-25%" value="1.0pF"/>
-<part name="C9" library="SparkFun-Capacitors" deviceset="1.0PF" device="-0603-50V-25%" value="1.0pF"/>
+<part name="C8" library="SparkFun-Capacitors" deviceset="1.0PF" device="-0603-50V-25%" value="DNP">
+<attribute name="PROD_ID" value=""/>
+</part>
+<part name="C9" library="SparkFun-Capacitors" deviceset="1.0PF" device="-0603-50V-25%" value="DNP">
+<attribute name="PROD_ID" value=""/>
+</part>
 <part name="GND20" library="SparkFun-PowerSymbols" deviceset="GND" device=""/>
 <part name="GND21" library="SparkFun-PowerSymbols" deviceset="GND" device=""/>
