File: Production/SparkFun_Simultaneous_RFID_Reader_M7E-Panel.brd (EAGLE design)
At the start: 121.4 x 210.8 mm, 681 parts, among them J10 U.FL, J14 U.FL, J18 U.FL, J22 U.FL, J26 U.FL, J30 U.FL, J34 U.FL, J5 U.FL, J6 U.FL, U1 UHF_RFID_NANO_MODULE_M7E_HECTO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

Commit message: Fix DNP components and PROD_ID values
Parts:
- C1, C10, C14, C17, C18, C19, C23, C26, C27, C28, C32, C35, C36, C37, C41, C44, C45, C46, C5, C50, C53, C54, C55, C59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: value 1.0pF -> DNP
